File: YMFC-32-kicad/YMFC-32.kicad_sch (KiCad schematic)
At the start: 23 parts, among them J1 RECEIVER, J10 MPU6050, J11 MS5611, J12 COMPASS, J2 M1, J3 M2, J4 M3, J5 M4, J6 VCC_BAT, J7 TELEMETRY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

Commit message: clean files
Parts:
- J2: value M1 -> MOTOR_1
- J3: value M2 -> MOTOR_2
- J4: value M3 -> MOTOR_3
- J5: value M4 -> MOTOR_4
- J6: footprint Connector_PinHeader_2.54mm:PinHeader_1x01_P2.54mm_Vertical -> TestPoint:TestPoint_Pad_4.0x4.0mm
- U1: footprint bluepill:YAAJ_BluePill_SWD_1 -> bluepill:YAAJ_BluePill_1
