File: YMFC-32-kicad/YMFC-32.kicad_pcb (KiCad board)
At the start: 2 copper layers, 80 x 80 mm, 23 parts, among them J1 RECEIVER, J10 MPU6050, J11 MS5611, J12 COMPASS, J2 MOTOR 1, J3 MOTOR 2, J4 MOTOR 3, J5 MOTOR 4, J6 VCC_BAT, J7 TELEMETRY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

Commit message: clean files
Parts:
- J10: footprint Connector_PinSocket_2.54mm:PinSocket_1x08_P2.54mm_Vertical -> Connector_PinHeader_2.54mm:PinHeader_1x08_P2.54mm_Vertical
- J11: footprint Connector_PinSocket_2.54mm:PinSocket_1x07_P2.54mm_Vertical -> Connector_PinHeader_2.54mm:PinHeader_1x07_P2.54mm_Vertical
- J12: footprint Connector_PinSocket_2.54mm:PinSocket_1x05_P2.54mm_Vertical -> Connector_PinHeader_2.54mm:PinHeader_1x05_P2.54mm_Vertical

Commit message: rev1
Parts:
- moved J10 19.4 mm to (111.5, 83.4), turned to 90 degrees
Routing:
- net +5V: track 166.4 -> 194.4 mm, vias 3 -> 5
- net GND1: track 118.3 -> 132.7 mm, vias 4 -> 6
- net SCL: track 128.1 -> 136.0 mm, vias 0 -> 1
- net +3V3: track 122.5 -> 125.9 mm, vias 3 -> 7
- net SDA: track 105.5 -> 103.9 mm, vias 1 -> 3
Other:
- board text added: "YMFC-32 rev1"
- board text removed: "YMFC-32 rev0"
